File: hw/board/board.kicad_sch (KiCad schematic)
At the start: 1 part

Commit message: Create board
Parts:
- added D1: LED, LED_SMD:LED_0805_2012Metric, symbol Device:LED
- added R1: 100, Resistor_SMD:R_0805_2012Metric, symbol Device:R
- added U1: W65C02S, Package_DIP:DIP-40_W15.24mm_LongPads, symbol 65xx:W65C02S
- J1: renamed from J?; footprint Connector_PinHeader_2.54mm:PinHeader_2x20_P2.54mm_Vertical -> Connector_PinSocket_2.54mm:PinSocket_2x20_P2.54mm_Vertical
Connections:
- net at J1.1 (Pin_1): now also D1.1 (K)
- net ~{NMIB}: now reaches J1.10 (Pin_10)
- net ~{NMIB}: now also U1.6 (~{NMIB})
- net +5V: now reaches J1.11 (Pin_11)
- net GND: now reaches J1.12 (Pin_12)
- net GND: now also J1.30 (Pin_30), U1.21 (VSS)
- net R~{WB}: now reaches J1.13 (Pin_13)
- net R~{WB}: now also U1.34 (R~{WB})
- net SYNC: now reaches J1.14 (Pin_14)
- net SYNC: now also U1.7 (SYNC)
- net D0: now reaches J1.15 (Pin_15)
- net D0: now also U1.33 (D0)
- net A0: now reaches J1.16 (Pin_16)
- net A0: now also U1.9 (A0)
- net D1: now reaches J1.17 (Pin_17)
- net D1: now also U1.32 (D1)
- net A1: now reaches J1.18 (Pin_18)
- net A1: now also U1.10 (A1)
- net D2: now reaches J1.19 (Pin_19)
- net D2: now also U1.31 (D2)
- net VPB: now reaches J1.2 (Pin_2)
- net VPB: now also U1.1 (VPB)
- net A2: now reaches J1.20 (Pin_20)
- net A2: now also U1.11 (A2)
- net D3: now reaches J1.21 (Pin_21)
- net D3: now also U1.30 (D3)
- net A3: now reaches J1.22 (Pin_22)
- net A3: now also U1.12 (A3)
- net D4: now reaches J1.23 (Pin_23)
- net D4: now also U1.29 (D4)
- net A4: now reaches J1.24 (Pin_24)
- net A4: now also U1.13 (A4)
- net D5: now reaches J1.25 (Pin_25)
- net D5: now also U1.28 (D5)
- net A5: now reaches J1.26 (Pin_26)
- net A5: now also U1.14 (A5)
- net D6: now reaches J1.27 (Pin_27)
- net D6: now also U1.27 (D6)
- net A6: now reaches J1.28 (Pin_28)
- net A6: now also U1.15 (A6)
- net +3V3: now reaches J1.29 (Pin_29)
- net +3V3: now also R1.1, U1.8 (VDD)
- net ~{RESB}: now reaches J1.3 (Pin_3)
- net ~{RESB}: now also U1.40 (~{RESB})
- net D7: now reaches J1.31 (Pin_31)
- net D7: now also U1.26 (D7)
- net A7: now reaches J1.32 (Pin_32)
- net A7: now also U1.16 (A7)
- net A15: now reaches J1.33 (Pin_33)
- net A15: now also U1.25 (A15)
- net A8: now reaches J1.34 (Pin_34)
- net A8: now also U1.17 (A8)
- net A14: now reaches J1.35 (Pin_35)
- net A14: now also U1.24 (A14)
- net A9: now reaches J1.36 (Pin_36)
- net A9: now also U1.18 (A9)
- net A13: now reaches J1.37 (Pin_37)
- net A13: now also U1.23 (A13)
- net A10: now reaches J1.38 (Pin_38)
- net A10: now also U1.19 (A10)
- net A12: now reaches J1.39 (Pin_39)
- net A12: now also U1.22 (A12)
- net RDY: now reaches J1.4 (Pin_4)
- net RDY: now also U1.2 (RDY)
- net A11: now reaches J1.40 (Pin_40)
- net A11: now also U1.20 (A11)
- net ~{SOB}: now reaches J1.5 (Pin_5)
- net ~{SOB}: now also U1.38 (~{SOB})
- net ~{IRQB}: now reaches J1.6 (Pin_6)
- net ~{IRQB}: now also U1.4 (~{IRQB})
- net PHI2: now reaches J1.7 (Pin_7)
- net PHI2: now also U1.37 (PHI2)
- net ~{MLB}: now reaches J1.8 (Pin_8)
- net ~{MLB}: now also U1.5 (~{MLB})
- net BE: now reaches J1.9 (Pin_9)
- net BE: now also U1.36 (BE)
- new net: D1.2 (A), R1.2
- no-connect marks 0 -> 2

Commit message: add basic stuff to board
Parts:
- removed D1: LED, LED_SMD:LED_0805_2012Metric, symbol Device:LED
- removed J1: Conn_02x20_Odd_Even, Connector_PinSocket_2.54mm:PinSocket_2x20_P2.54mm_Vertical, symbol Connector_Generic:Conn_02x20_Odd_Even
- removed U1: W65C02S, Package_DIP:DIP-40_W15.24mm_LongPads, symbol 65xx:W65C02S
- added C1, C23, C24, C25, C26, C27, C29, C30, C31, C32: (no value), symbol Device:C
- added C10, C11, C12, C13, C28, C33, C34, C35: (no value), symbol Device:C_Small
- added C14, C15, C17, C18, C19, C20, C22: 100n, symbol Device:C_Small
- added C16, C21: 4.7u, symbol Device:C_Small
- added C2, C3, C4, C5, C6, C7, C8, C9: 100n, symbol Device:C
- added J1: (no value), symbol Connector:USB_C_Receptacle_USB2.0
- added L1, L3: (no value), symbol Device:L
- added L2: 600R @ 100MHz, symbol Device:L
- added R10: 10k, symbol Device:R
- added R11, R12, R2, R3, R4, R5, R6, R7, R8, R9: (no value), symbol Device:R
- added U1: (no value), symbol IC:T8Q144
- added U2: (no value), symbol Regulator_Linear:LD1117S33TR_SOT223
- added U3: (no value), symbol Regulator_Linear:LD1117S12TR_SOT223
- added U4: (no value), symbol Interface_USB:FT2232HL
- added U5: (no value), symbol Memory_EEPROM:93LCxxBxxOT
- added Y1: (no value), symbol Device:Crystal
- R1: value 100 -> (none); footprint Resistor_SMD:R_0805_2012Metric -> (none)
Connections:
- net +3V3: now also C16.1, C17.1, C18.1, C19.1, C20.1, C27.1, C28.1, C29.1, C33.1, L1.1, L2.1, R10.2, R3.2, R5.2, R6.1, R7.1, R8.1, U1.12 (VCCIO_1C_1D), U1.122 (VCCIO_3A), U1.143 (VCCIO_1E), U1.21 (VCCIO_1B), U1.23 (VCCIO_1A), U1.51 (VCCIO_4B), U1.52 (VCCIO_4B), U1.62 (VCCIO_4A), U1.63 (VCCIO_4A), U1.88 (VCCIO_3E), U1.91 (VCCIO_3D), U1.95 (VCCIO_3B_3C), U2.2 (VO), U3.3 (VI), U4.20 (VCCIO), U4.31 (VCCIO), U4.42 (VCCIO), U4.50 (VREGIN), U4.56 (VCCIO), U5.6 (VCC); no longer R1.1
- net +5V: now also C25.1, C26.1, J1.A4 (VBUS), J1.A9 (VBUS), J1.B4 (VBUS), J1.B9 (VBUS), R11.2, U2.3 (VI)
- net GND: now also R1.2, C1.2, C10.2, C11.2, C12.2, C13.2, C14.2, C15.2, C16.2, C17.2, C18.2, C19.2, C2.2, C20.2, C21.2, C22.2, C23.2, C24.2, C25.2, C26.2, C27.2, C28.2, C29.2, C3.2, C30.2, C31.2, C32.2, C33.2, C34.1, C35.1, C4.2, C5.2, C6.2, C7.2, C8.2, C9.2, J1.A1 (GND), J1.A12 (GND), J1.B1 (GND), J1.B12 (GND), J1.S1 (SHIELD), R12.2, R2.2, R4.1, U1.1 (GND), U1.104 (GND), U1.108 (GND), U1.120 (GND), U1.121 (GND), U1.126 (GND), U1.127 (GND), U1.129 (GND), U1.133 (GND), U1.37 (GND), U1.44 (GND), U1.5 (GND), U1.50 (GND), U1.64 (GND), U1.9 (GND), U1.94 (GND), U2.1 (GND), U3.1 (GND), U4.1 (GND), U4.10 (AGND), U4.11 (GND), U4.13 (TEST), U4.15 (GND), U4.25 (GND), U4.35 (GND), U4.47 (GND), U4.5 (GND), U4.51 (GND), U5.2 (GND)
- new net: C34.2, U4.2 (OSCI), Y1.2
- new net: R3.1, U4.28 (ACBUS2)
- new net: C35.2, U4.3 (OSCO), Y1.1
- new net: R10.1, U4.53 (BCBUS2)
- new net: R11.1, R12.1, U4.59 (BCBUS7)
- new net: R4.2, U4.6 (REF)
- new net: R6.2, R9.2, U4.61 (EEDATA), U5.3 (DI)
- new net: R7.2, U4.62 (EECLK), U5.4 (CLK)
- new net: R8.2, U4.63 (EECS), U5.5 (CS)
- new net: C23.1, C24.1, L3.2, U1.107 (VCCA_TR), U1.2 (VCCA_TL), U1.73 (VCCA_BR)
- new net: J1.A5 (CC1), R1.1
- new net: J1.B5 (CC2), R2.1
- new net: R9.1, U5.1 (DO)
- new net +1V2: C1.1, C2.1, C3.1, C30.1, C31.1, C32.1, C4.1, C5.1, C6.1, C7.1, C8.1, C9.1, L3.1, U1.125 (VCC), U1.128 (VCC), U1.13 (VCC), U1.130 (VCC), U1.22 (VCC), U1.49 (VCC), U1.57 (VCC), U1.85 (VCC), U1.96 (VCC), U3.2 (VO)
- new net CDONE: U4.22 (ADBUS5)
- new net CRESET_B: U4.21 (ADBUS4)
- new net FT_RST: R5.1, U4.14 (~{RESET})
- new net HOLD: U4.23 (ADBUS6)
- new net SPI_CLK: U4.16 (ADBUS0)
- new net SPI_MISO: U4.18 (ADBUS2)
- new net SPI_MOSI: U4.17 (ADBUS1)
- new net SPI_SS: U4.19 (ADBUS3)
- new net TCK: U4.38 (BDBUS0)
- new net TDI: U4.39 (BDBUS1)
- new net TDO: U4.40 (BDBUS2)
- new net TMS: U4.41 (BDBUS3)
- new net USB_N: J1.A7 (D-), J1.B7 (D-), U4.7 (DM)
- new net USB_P: J1.A6 (D+), J1.B6 (D+), U4.8 (DP)
- new net VPHY: C21.1, C22.1, L2.2, U4.4 (VPHY)
- new net VPLL: C10.1, C11.1, L1.2, U4.9 (VPLL)
- new net VRO: C12.1, C13.1, C14.1, C15.1, U4.12 (VCORE), U4.37 (VCORE), U4.49 (VREGOUT), U4.64 (VCORE)
- no-connect marks 2 -> 20
