File: hw/efinix_shield/efinix_shield.kicad_sch (KiCad schematic)
At the start: 14 parts, among them J1 DB15_Female_HighDensity_Mount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, U1 T20BGA256_DEV_GPIO_1D1E, U2 T20BGA256_DEV_GPIO_1B1C, U3 T20BGA256_DEV_GPIO_3

Commit message: Redo shield, removing FPGA
Don't have the FPGA on the shield, just have it be a board that plugs
into the FPGA.

Don't mind the component and footprint choices yet, I still need to
figure out exactly which parts to use.
Parts:
- removed J?: SD_Card, symbol Connector:SD_Card
- removed J?: Micro_SD_Card, symbol Connector:Micro_SD_Card
- removed U1: T20BGA256_DEV_GPIO_1D1E, Connector_PinSocket_2.54mm:PinSocket_2x18_P2.54mm_Vertical, symbol Header:T20BGA256_DEV_GPIO_1D1E
- removed U2: T20BGA256_DEV_GPIO_1B1C, Connector_PinSocket_2.54mm:PinSocket_2x18_P2.54mm_Vertical, symbol Header:T20BGA256_DEV_GPIO_1B1C
- removed U3: T20BGA256_DEV_GPIO_3, Connector_PinSocket_2.54mm:PinSocket_2x16_P2.54mm_Vertical, symbol Header:T20BGA256_DEV_GPIO_3
- added J2: SD_Card, symbol Connector:SD_Card
- added J3: Conn_02x18_Odd_Even, Connector_PinSocket_2.54mm:PinSocket_2x18_P2.54mm_Vertical, symbol Connector_Generic:Conn_02x18_Odd_Even
- added J4: Micro_SD_Card, symbol Connector:Micro_SD_Card
- added U1: MAX3421E, Package_QFP:LQFP-32_5x5mm_P0.5mm, symbol IC:MAX3421E
- added U2: CP2102N-Axx-xQFN24, Package_DFN_QFN:QFN-24-1EP_4x4mm_P0.5mm_EP2.6x2.6mm, symbol Interface_USB:CP2102N-Axx-xQFN24
- J1: footprint (none) -> Connector_Dsub:DSUB-15-HD_Male_Horizontal_P2.29x1.98mm_EdgePinOffset3.03mm_Housed_MountingHolesOffset4.94mm
- R1, R2: footprint (none) -> Resistor_SMD:R_0603_1608Metric_Pad0.98x0.95mm_HandSolder
- RN1, RN2, RN3, RN4, RN5, RN6: footprint (none) -> Resistor_SMD:R_Array_Concave_4x0402
Connections:
- net +3V3: now also J2.4 (VDD), J4.4 (VDD)
- net GND: now also J2.12 (SHELL1), J2.13 (SHELL2), J2.3 (VSS), J2.6 (VSS), J3.34 (Pin_34), J3.35 (Pin_35), J3.36 (Pin_36), J4.6 (VSS), J4.9 (SHIELD)
- net SD_CLK: now also J2.5 (CLK), J4.5 (CLK)
- net SD_CMD: now also J2.2 (CMD), J4.3 (CMD)
- net SD_DAT0: now also J2.7 (DAT0), J4.7 (DAT0)
- net SD_DAT1: now also J2.8 (DAT1), J4.8 (DAT1)
- net SD_DAT2: now also J2.9 (DAT2), J4.1 (DAT2)
- net SD_DAT3: now also J2.1 (CD/DAT3), J4.2 (DAT3/CD)
- new net: U2.2 (GND), U2.25 (GND)
- new net VDD: J3.1 (Pin_1), J3.2 (Pin_2)

Commit message: Start over pretty much.
Parts:
- removed J4: Micro_SD_Card, symbol Connector:Micro_SD_Card
- J1: value DB15_Female_HighDensity_MountingHoles -> VGA; footprint Connector_Dsub:DSUB-15-HD_Male_Horizontal_P2.29x1.98mm_EdgePinOffset3.03mm_Housed_MountingHolesOffset4.94mm -> Connector_Dsub:ICD15S13E4GX00LF; Link (none) -> https://www.digikey.com/en/products/detail/amphenol-cs-fci/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; Part Name (none) -> ICD15S13E4GX00LF

Commit message: throw some stuff on.
This will have to be changed, some things like the VGA connector will
not work because they will interfere with the cpu adapter.

It may be worth thinking about making these smaller and not including
the ethernet for example, since that will not come for a while.

The only things we really need to start are the SD card and serial port.
Parts:
- removed J1: VGA, Connector_Dsub:ICD15S13E4GX00LF, symbol Connector:DB15_Female_HighDensity_MountingHoles
- removed J2: SD_Card, symbol Connector:SD_Card
- removed R1, R2: 120, Resistor_SMD:R_0603_1608Metric_Pad0.98x0.95mm_HandSolder, symbol Device:R
- removed RN1, RN2, RN5: 1k, Resistor_SMD:R_Array_Concave_4x0402, symbol Device:R_Pack04
- removed RN3, RN4, RN6: 2k, Resistor_SMD:R_Array_Concave_4x0402, symbol Device:R_Pack04
- added C1001, C1002: 0.1u, Capacitor_SMD:C_0603_1608Metric_Pad1.08x0.95mm_HandSolder, symbol Device:C
- added C1003: 10u, Capacitor_SMD:C_0603_1608Metric_Pad1.08x0.95mm_HandSolder, symbol Device:C
- added D1001: 1N4148, Diode_SMD:D_0603_1608Metric_Pad1.05x0.95mm_HandSolder, symbol Device:D
- added J1001: USB_B_Mini, Connector_USB:USB_Mini-B_Wuerth_65100516121_Horizontal, symbol Connector:USB_B_Mini
- added J1002: USB_A, Connector_USB:FCI_87520-0010BLF, symbol Connector:USB_A
- added J1004: 10067847-001RLF, Connector_Card:AMPHENOL_10067847-001RLF, symbol Connector:10067847-001RLF
- added J1005: JX0011D21NL, Connector_RJ:JX0011D21NL, symbol Connector:JX0011D21NL
- added R1001: 4k7, Resistor_SMD:R_0603_1608Metric_Pad0.98x0.95mm_HandSolder, symbol Device:R
- added R1002: 10k, Resistor_SMD:R_0603_1608Metric_Pad0.98x0.95mm_HandSolder, symbol Device:R
- added R1003: 220, Resistor_SMD:R_0603_1608Metric_Pad0.98x0.95mm_HandSolder, symbol Device:R
- added R1004: 6.49k 1%, Resistor_SMD:R_0603_1608Metric_Pad0.98x0.95mm_HandSolder, symbol Device:R
- added R1005: 1k, Resistor_SMD:R_0603_1608Metric_Pad0.98x0.95mm_HandSolder, symbol Device:R
- added U1003: KSZ8081RNA, Package_DFN_QFN:QFN-24-1EP_4x4mm_P0.5mm_EP2.6x2.6mm, symbol Interface_Ethernet:KSZ8081RNA
- renumbered J3 to J1003, U1 to U1001, U2 to U1002
Connections:
- net VDD is gone; now on net +3V3: J1003.1 (Pin_1), J1003.2 (Pin_2)
- net +3V3: now also U1001.23 (VCC), D1001.2 (A), J1004.4 (VDD), R1001.1, R1002.1, R1003.1, U1003.14 (VDDIO), U1003.2 (VDDA_3.3)
- net GND: now also U1001.19 (GND), U1001.3 (GND), U1002.2 (GND), U1002.25 (GND), C1001.1, C1002.1, C1003.2, J1004.3 (VSS), J1004.6 (VSS), J1004.G1 (GND), J1004.G2 (GND), J1005.8 (GND), R1004.2, R1005.2, U1003.22 (GND), U1003.25 (GND)
- net VGA_BLUE_0: now also J1003.24 (Pin_24)
- net VGA_BLUE_1: now also J1003.26 (Pin_26)
- net VGA_BLUE_2: now also J1003.27 (Pin_27)
- net VGA_GREEN_0: now also J1003.28 (Pin_28)
- net VGA_GREEN_1: now also J1003.29 (Pin_29)
- net VGA_GREEN_2: now also J1003.30 (Pin_30)
- net VGA_HS: now also J1003.22 (Pin_22)
- net VGA_RED_0: now also J1003.31 (Pin_31)
- net VGA_RED_1: now also J1003.32 (Pin_32)
- net VGA_RED_2: now also J1003.33 (Pin_33)
- net VGA_VS: now also J1003.21 (Pin_21)
- net RMII_RXD0: now reaches J1003.10 (Pin_10)
- net RMII_RXD0: now also U1003.13 (RXD0)
- net RMII_RXD1: now reaches J1003.11 (Pin_11)
- net RMII_RXD1: now also U1003.12 (RXD1)
- net MDCLK: now reaches J1003.12 (Pin_12)
- net MDCLK: now also U1003.11 (MDC)
- net MDIO: now reaches J1003.13 (Pin_13)
- net MDIO: now also U1003.10 (MDIO)
- net UART_RX: now reaches J1003.14 (Pin_14)
- net UART_RX: now also U1002.21 (TXD)
- net UART_TX: now reaches J1003.15 (Pin_15)
- net UART_TX: now also U1002.20 (RXD)
- net SPI_USB_CS: now reaches J1003.16 (Pin_16)
- net SPI_USB_CS: now also U1001.14 (~{SS})
- net SPI_MISO: now reaches J1003.17 (Pin_17)
- net SPI_MISO: now also U1001.15 (MISO), J1004.7 (DAT0)
- net SPI_CLK: now reaches J1003.18 (Pin_18)
- net SPI_CLK: now also U1001.13 (SCLK), J1004.5 (CLK)
- net SPI_MOSI: now reaches J1003.19 (Pin_19)
- net SPI_MOSI: now also U1001.16 (MOSI), J1004.2 (CMD)
- net SPI_SD_CS: now reaches J1003.20 (Pin_20)
- net SPI_SD_CS: now also J1004.1 (DAT3/CD)
- net DVI_DE: now reaches J1003.23 (Pin_23)
- net DVI_CLK: now reaches J1003.25 (Pin_25)
- net DVI_CLK: now also U1003.8 (XI)
- net SPI_CS_3: now reaches J1003.3 (Pin_3)
- net RMII_TXD1: now reaches J1003.4 (Pin_4)
- net RMII_TXD1: now also U1003.21 (TXD1)
- net RMII_TXD0: now reaches J1003.5 (Pin_5)
- net RMII_TXD0: now also U1003.20 (TXD0)
- net RMII_TX_EN: now reaches J1003.6 (Pin_6)
- net RMII_TX_EN: now also U1003.19 (TXEN)
- net RMII_RX_ERR: now reaches J1003.7 (Pin_7)
- net RMII_RX_ERR: now also U1003.17 (RXER)
- net RMII_CLK_REF: now reaches J1003.8 (Pin_8)
- net RMII_CLK_REF: now also U1003.16 (REF_CLK)
- net RMII_CRS_DV: now reaches J1003.9 (Pin_9)
- net RMII_CRS_DV: now also U1003.15 (CRS_DV/PHYAD[1:0])
- new net: J1005.9 (L+), R1003.2
- new net: J1005.10 (L-), R1001.2, R1005.1, U1003.23 (LED0/ANEN_SPEED)
- new net: R1004.1, U1003.9 (REXT)
- new net: C1002.2, J1005.4 (CT)
- new net: C1001.2, J1005.5 (CT)
- new net +1V2: U1003.1 (VDD_1.2)
- new net RX+: J1005.3 (RD+), U1003.4 (RXP)
- new net RX-: J1005.6 (RD-), U1003.3 (RXM)
- new net TX+: J1005.1 (TD+), U1003.6 (TXP)
- new net TX-: J1005.2 (TD-), U1003.5 (TXM)
- new net ~{PHY_RST}: C1003.1, D1001.1 (K), R1002.2, U1003.24 (~{RST})
- no-connect marks 19 -> 8
Other:
- added sheet video (video.kicad_sch)
- note added: "100mpbs"
- note added: "10mbps"
- moved on the sheet: J1003, U1001, U1002

Commit message: Start work on simpler board
Parts:
- removed D1001: 1N4148, Diode_SMD:D_0603_1608Metric_Pad1.05x0.95mm_HandSolder, symbol Device:D
- removed J1005: JX0011D21NL, Connector_RJ:JX0011D21NL, symbol Connector:JX0011D21NL
- removed U1002: CP2102N-Axx-xQFN24, Package_DFN_QFN:QFN-24-1EP_4x4mm_P0.5mm_EP2.6x2.6mm, symbol Interface_USB:CP2102N-Axx-xQFN24
- removed U1003: KSZ8081RNA, Package_DFN_QFN:QFN-24-1EP_4x4mm_P0.5mm_EP2.6x2.6mm, symbol Interface_Ethernet:KSZ8081RNA
- added C1004, C1005: C, Capacitor_SMD:C_0805_2012Metric_Pad1.18x1.45mm_HandSolder, symbol Device:C
- added D1001: RED, LED_SMD:LED_0805_2012Metric_Pad1.15x1.40mm_HandSolder, symbol Device:LED
- added D1002: GRN, LED_SMD:LED_0805_2012Metric_Pad1.15x1.40mm_HandSolder, symbol Device:LED
- added R1006, R1007: 33, Resistor_SMD:R_0805_2012Metric_Pad1.20x1.40mm_HandSolder, symbol Device:R
- added U1001: CP2102N-Axx-xQFN24, Package_DFN_QFN:QFN-24-1EP_4x4mm_P0.5mm_EP2.6x2.6mm, symbol Interface_USB:CP2102N-Axx-xQFN24
- added Y1001: 12MHz, Crystal:Crystal_HC49-U_Vertical, symbol Device:Crystal
- C1001: value 0.1u -> 1u; footprint Capacitor_SMD:C_0603_1608Metric_Pad1.08x0.95mm_HandSolder -> Capacitor_SMD:C_0805_2012Metric_Pad1.18x1.45mm_HandSolder
- C1002: footprint Capacitor_SMD:C_0603_1608Metric_Pad1.08x0.95mm_HandSolder -> Capacitor_SMD:C_0805_2012Metric_Pad1.18x1.45mm_HandSolder
- C1003: value 10u -> 4.7u; footprint Capacitor_SMD:C_0603_1608Metric_Pad1.08x0.95mm_HandSolder -> Capacitor_SMD:C_0805_2012Metric_Pad1.18x1.45mm_HandSolder
- R1001: value 4k7 -> 10k; footprint Resistor_SMD:R_0603_1608Metric_Pad0.98x0.95mm_HandSolder -> Resistor_SMD:R_0805_2012Metric_Pad1.20x1.40mm_HandSolder
- R1002, R1005: footprint Resistor_SMD:R_0603_1608Metric_Pad0.98x0.95mm_HandSolder -> Resistor_SMD:R_0805_2012Metric_Pad1.20x1.40mm_HandSolder
- R1003: value 220 -> 10k; footprint Resistor_SMD:R_0603_1608Metric_Pad0.98x0.95mm_HandSolder -> Resistor_SMD:R_0805_2012Metric_Pad1.20x1.40mm_HandSolder
- R1004: value 6.49k 1% -> 1k; footprint Resistor_SMD:R_0603_1608Metric_Pad0.98x0.95mm_HandSolder -> Resistor_SMD:R_0805_2012Metric_Pad1.20x1.40mm_HandSolder
- renumbered J1003 to J1001, J1001 to J1002, J1002 to J1003, U1001 to U1002
Connections:
- net DVI_CLK is gone; now on net VGA_BLUE_0: J1001.25 (Pin_25)
- net DVI_DE is gone; now on net VGA_HS: J1001.23 (Pin_23)
- net +3V3: now also C1001.1, C1002.1, R1004.1, R1005.1, U1002.2 (VL), U1001.5 (VIO), U1001.6 (VDD), U1001.7 (VREGIN); no longer R1001.1, R1002.1, R1003.1
- net GND: now also C1001.2, C1002.2, J1002.5 (GND), J1002.6 (Shield), J1003.4 (GND), J1003.5 (Shield), R1003.2, C1004.2, C1005.2, U1001.2 (GND), U1001.25 (GND); no longer C1001.1, C1002.1, R1004.2, R1005.2
- net SPI_CLK: now also J1001.21 (Pin_21); no longer J1001.18 (Pin_18), J1004.5 (CLK)
- net SPI_CS_3: no longer J1001.3 (Pin_3)
- net SPI_MISO: now also J1001.19 (Pin_19); no longer J1001.17 (Pin_17), J1004.7 (DAT0)
- net SPI_MOSI: now also J1001.18 (Pin_18); no longer J1001.19 (Pin_19), J1004.2 (CMD)
- net SPI_USB_CS: now also J1001.20 (Pin_20); no longer J1001.16 (Pin_16)
- net UART_RX: now also U1001.21 (TXD)
- net UART_TX: now also U1001.20 (RXD)
- net VGA_BLUE_0: no longer J1001.24 (Pin_24)
- net VGA_HS: no longer J1001.22 (Pin_22)
- net VGA_VS: now also J1001.24 (Pin_24); no longer J1001.21 (Pin_21)
- net at R1001.2: now also R1002.1, U1001.8 (VBUS); no longer R1005.1
- net ~{RESET}: now reaches U1002.12 (~{RES})
- net ~{RESET}: now also J1001.22 (Pin_22), U1001.9 (~{RST})
- net USB_GPX: now reaches U1002.17 (GPX)
- net USB_GPX: now also J1001.17 (Pin_17)
- net USB_INT: now reaches U1002.18 (INT)
- net USB_INT: now also J1001.16 (Pin_16)
- net at U1002.20 (D-): now also R1006.1
- net at U1002.21 (D+): now also R1007.2
- net at U1002.24 (XI): now also C1004.1, Y1001.1
- net at U1002.25 (XO): now also C1005.1, Y1001.2
- net SD_D1: now reaches J1004.8 (DAT1)
- net SD_D2: now reaches J1004.9 (DAT2)
- net +5V: now reaches J1003.1 (VBUS)
- net +5V: now also C1003.1, J1002.1 (VBUS), R1001.1
- net at J1003.2 (D-): now also R1006.2
- net at J1003.3 (D+): now also R1007.1
- net USBB_DN: now reaches J1002.2 (D-)
- net USBB_DN: now also U1001.4 (D-)
- net USBB_DP: now reaches J1002.3 (D+)
- net USBB_DP: now also U1001.3 (D+)
- net MDCLK: no longer names the net of J1001.12 (Pin_12)
- net MDIO: no longer names the net of J1001.13 (Pin_13)
- net RMII_CLK_REF: no longer names the net of J1001.8 (Pin_8)
- net RMII_CRS_DV: no longer names the net of J1001.9 (Pin_9)
- net RMII_RXD0: no longer names the net of J1001.10 (Pin_10)
- net RMII_RXD1: no longer names the net of J1001.11 (Pin_11)
- net RMII_RX_ERR: no longer names the net of J1001.7 (Pin_7)
- net RMII_TXD0: no longer names the net of J1001.5 (Pin_5)
- net RMII_TXD1: no longer names the net of J1001.4 (Pin_4)
- net RMII_TX_EN: no longer names the net of J1001.6 (Pin_6)
- net SPI_SD_CS renamed SD_D3
- net SD_D3: no longer J1001.20 (Pin_20)
- net ~{PHY_RST}: no longer names the net of R1002.2
- net ~{PHY_RST}: now also R1003.1; no longer C1003.1
- new net: D1001.2 (A), R1004.2
- new net: D1002.2 (A), R1005.2
- new net RX_LED: D1002.1 (K), U1001.13 (~{RXT}/GPIO.1)
- new net SD_CLK: J1004.5 (CLK)
- new net SD_CMD: J1004.2 (CMD)
- new net SD_D0: J1004.7 (DAT0)
- new net TX_LED: D1001.1 (K), U1001.14 (~{TXT}/GPIO.0)
- no-connect marks 8 -> 14
Other:
- sheet video ports: added none; removed DVI_CLK, DVI_DE
- note removed: "100mpbs"
- note removed: "10mbps"
- moved on the sheet: J1002, J1003, J1004, U1002

Commit message: Finish routing sd card slot, update gitignore
Parts:
- added J1001: Conn_01x06, Connector_PinHeader_2.54mm:PinHeader_1x06_P2.54mm_Vertical, symbol Connector_Generic:Conn_01x06
- added R1001, R1003: 0, Resistor_SMD:R_0805_2012Metric_Pad1.20x1.40mm_HandSolder, symbol Device:R
- added R1002, R1004, R1005: 10k, Resistor_SMD:R_0805_2012Metric_Pad1.20x1.40mm_HandSolder, symbol Device:R
- renumbered J1001 to J1002, J1002 to J1003, J1003 to J1004, J1004 to J1005, R1001 to R1006, R1002 to R1007, R1003 to R1008, R1004 to R1009, R1005 to R1010, R1006 to R1011, R1007 to R1012
Connections:
- net +5V: now also R1001.1
- net GND: now also J1001.1 (Pin_1), R1005.2
- net SD_CLK: now also J1002.10 (Pin_10)
- net SD_CMD: now also J1002.11 (Pin_11)
- net SD_D0: now also J1002.9 (Pin_9)
- net SD_D1: now also J1002.8 (Pin_8)
- net SD_D2: now also J1002.13 (Pin_13)
- net SD_D3: now also J1002.12 (Pin_12)
- net UART_RX: now also R1002.1
- net UART_TX: now also R1003.1
- new net: J1001.3 (Pin_3), R1001.2
- new net: R1004.2, R1005.1
- new net HOST_RX: J1001.5 (Pin_5), R1003.2
- new net HOST_TX: J1001.4 (Pin_4), R1002.2, R1004.1
- no-connect marks 14 -> 16
