File: hw/efinix_board/cpu.kicad_sch (KiCad schematic)
At the start: 8 parts, among them U501 W65C02SQ

Commit message: More routing
Connections:
- net at U501.33 (NC): no longer U501.6 (NC)
- no-connect marks 3 -> 4
Changed lines of the file:
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@@
   (no_connect (at 130.81 69.85))
   (no_connect (at 130.81 67.31))
-  (no_connect (at 156.21 49.53))
+  (no_connect (at 142.24 115.57))
+  (no_connect (at 144.78 115.57))
   (bus_entry (at 165.1 59.69) (size 2.54 2.54)
     (stroke (width 0) (type default) (color 0 0 0 0))
