File: hw/efinix_board/power.kicad_sch (KiCad schematic)
At the start: 55 parts, among them U1 T20F256, U2 TPS62826, U3 TPS62826

Commit message: Start working on sdram
Other:
- moved on the sheet: C37, C38, C39, C40, C41, C42, L2, L3, R2, R3, R4, R5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

Commit message: Update schematics and board
Parts:
- added R10, R8: 100k, Resistor_SMD:R_0402_1005Metric, symbol Device:R
- added R9: 33R, Resistor_SMD:R_0402_1005Metric, symbol Device:R
- added SW1: SW_Push, Button_Switch_THT:SW_1825966-1, symbol Switch:SW_Push
- added U5: ADM6713, Package_SC:ADM6711TAKSZ-REEL7, symbol Power_Supervisor:ADM6713
Connections:
- net +3V3: now also R10.1, R8.1, U5.4 (VCC)
- net GND: now also SW1.1, U5.1 (GND)
- new net: R9.2, SW1.2
- new net ~{CRESET}: R10.2, U5.2 (~{RST})
- new net ~{RST_REQ}: R8.2, R9.1, U5.3 (~{MR})
