File: hw/T120F484_dev/power.kicad_sch (KiCad schematic)
At the start: 1 part

Commit message: Do some work on clocks
Parts:
- removed U1: ~, symbol IC:T120F484
Other:
- note removed: "10uF/1uF per bank, alternate 0.1uF/0.01uF per pin"
- note removed: "18 Power pins 9 0.1uF, 9 0.01uF, per pin 2 10uF, 2 1uF, around outside"
- note removed: "22 power pins 11 0.1uF and 11 0.01uF, alternate per pin 4 10uF, 4 1uF, around outside of chip"
- note removed: "Resistor + ferrite + 1nf, 0.1uf/0.01uf per pin per each"
