File: hw/T120F484_dev/clock.kicad_sch (KiCad schematic)
At the start: 24 parts, among them J3 Conn_Coaxial, J4 Conn_Coaxial, J5 Conn_01x03, U4 Si5351A-B-GT, X1 25M, X2 50M, Y2 25M

Commit message: Update
Parts:
- U1: footprint (none) -> Package_BGA:BGA-484_22x22_18.0x18.0mm
Changed lines of the file:
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@@
 			)
 		)
-		(property "Datasheet" " ~"
+		(property "Datasheet" "~"
 			(at 227.33 132.08 0)
 			(effects
@@
 			)
 		)
-		(property "Datasheet" " ~"
+		(property "Datasheet" "~"
 			(at 227.33 101.6 0)
 			(effects
@@
 			)
 		)
-		(property "Footprint" ""
+		(property "Footprint" "Package_BGA:BGA-484_22x22_18.0x18.0mm"
 			(at 200.66 83.82 0)
 			(effects
