File: hw/T120F484_dev/config.kicad_sch (KiCad schematic)
At the start: 41 parts, among them J1 Conn_02x05_Odd_Even, J2 Conn_02x05_Odd_Even, Q1 Q_NPN_BEC, SW1 SW_Push, U2 MCP100-300D, U3 W25Q128JVS

Commit message: Update
Parts:
- U1: footprint (none) -> Package_BGA:BGA-484_22x22_18.0x18.0mm
Changed lines of the file:
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@@
 			)
 		)
-		(property "Footprint" ""
+		(property "Footprint" "Package_BGA:BGA-484_22x22_18.0x18.0mm"
 			(at 166.37 78.74 0)
 			(effects
