File: hw/T120F484_dev/ddr.kicad_sch (KiCad schematic)
At the start: 1 part

Commit message: Update
Parts:
- U1: footprint (none) -> Package_BGA:BGA-484_22x22_18.0x18.0mm
Changed lines of the file:
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@@
 			)
 		)
-		(property "Footprint" ""
+		(property "Footprint" "Package_BGA:BGA-484_22x22_18.0x18.0mm"
 			(at 11.43 67.31 0)
 			(effects
